File: PModCamera.kicad_pcb (KiCad board)
At the start: 2 copper layers, 40 x 45 mm, 19 parts, among them J1 Conn_01x24_MountingPin, J2 Conn_02x06_Odd_Even, J3 Conn_02x06_Odd_Even, U1 AMS1117-2.85, U2 AMS1117-1.5, X1 SG-5032CAN

Commit message: 修改等长线
Parts:
- moved C1 1.14 mm to (112.8, 105.9)
- moved C2 1.14 mm to (112.8, 107.4)
Connections:
- U1 pad 2: +2V8 -> +3V3
- U1 pad 3: +3V3 -> +2V8
Routing:
- net +3V3: track 58.9 -> 26.3 mm
- net /OV1_D6: track 20.9 -> 13.1 mm, vias 0 -> 1
- net /OV1_D4: track 20.7 -> 13.3 mm
- net /OV1_D2: track 20.8 -> 14.6 mm
- net /OV1_PWDN: track 34.8 -> 29.2 mm
- net /OV1_D5: track 20.8 -> 16.5 mm, vias 0 -> 1
- net /OV1_D7: track 20.8 -> 16.4 mm, vias 0 -> 1
- net /OV1_RESET: track 36.2 -> 32.0 mm
- net /OV1_D1: track 20.7 -> 17.3 mm
- net /OV1_SDA: track 40.0 -> 36.8 mm
- net /OV1_HREF: track 20.8 -> 18.0 mm
- net +2V8: track 68.2 -> 70.8 mm, vias 0 -> 2
- net GND: track 0.00 -> 1.98 mm, vias 6 -> 7
- net /OV1_VSYNC: track 20.8 -> 19.4 mm
- net /OV1_XCLK: track 30.2 -> 29.8 mm, vias 2 -> 0
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Other:
- board text added: "Designed By ARCW 2021.03.08 V1.2"
- board text removed: "Designed By ARCW 2020.12.28 V1.1"
